Commit message: tem changes

File: robot_descriptions/agibot_g1_with_gripper_description/agibot_g1_with_omnipicker.urdf (robot description, URDF)
Before this commit: robot agibot_g1_with_omni-picker, 52 links, 51 joints
Links:
- added link dummy_left_camera; visual box size=0.10 0.02 0.02
- added link left_camera_stand; visual mesh filename=package://agibot_g1_description/meshes/camera/omni_picker_c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
- added link right_camera_stand; visual mesh filename=package://agibot_g1_description/meshes/camera/omni_picker_c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
Joints:
- added joint left_camera_joint: type fixed, parent left_camera_stand, child dummy_left_camera, origin xyz=0 -0.07754 0.028618 rpy=0 -1.117 1.5708
- added joint left_camera_stand_joint: type fixed, parent left_end_link, child left_camera_stand, origin xyz=0 0 0.004
- added joint right_camera_stand_joint: type fixed, parent right_end_link, child right_camera_stand, origin xyz=0 0 0.004
- joint left_eef_joint: origin xyz=0.0 0.0 0.015 -> xyz=0.0 0.0 0.015 rpy=0 0 1.5707963267948966
- joint right_eef_joint: origin xyz=0.0 0.0 0.015 -> xyz=0.0 0.0 0.015 rpy=0 0 1.5707963267948966
